File: hw/car.kicad_sch (KiCad schematic)
At the start: 76 parts, among them J2 SWD, J31 TYPE-C-31-M-12, J61 aux-1, J61 aux-2, J61 aux-3, J61 batt-out, J61 btn, J61 display, J61 mot-l-a, J61 mot-l-b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

Commit message: плата - надписи
Connections:
- net a0: now reaches J61.2 (Pin_2), U11.14 (PA0)
- net a1: now reaches J61.3 (Pin_3), U11.15 (PA1)
- net a2: now reaches J61.2 (Pin_2), U11.16 (PA2)
- net a3: now reaches J61.3 (Pin_3), U11.17 (PA3)
- net a4: now reaches J61.4 (Pin_4), U11.20 (PA4)
- net c2: now reaches J61.3 (Pin_3), U11.10 (PC2)
- net c3: now reaches J61.4 (Pin_4), U11.11 (PC3)
- net c1: now reaches J61.2 (Pin_2), U11.9 (PC1)
Changed lines of the file:
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@@
+    (effects (font (size 1.27 1.27)) (justify left bottom))
+  )
+  (label "c3" (at 50.038 50.8 0) (fields_autoplaced)
     (effects (font (size 1.27 1.27)) (justify left bottom))
   )
@@
     (effects (font (size 1.27 1.27)) (justify left bottom))
   )
+  (label "a3" (at 122.682 34.29 0) (fields_autoplaced)
+    (effects (font (size 1.27 1.27)) (justify left bottom))
+  )
   (label "mot-l-flt" (at 211.582 26.416 0) (fields_autoplaced)
     (effects (font (size 1.27 1.27)) (justify left bottom))
@@
     (effects (font (size 1.27 1.27)) (justify left bottom))
   )
+  (label "a4" (at 122.682 36.83 0) (fields_autoplaced)
+    (effects (font (size 1.27 1.27)) (justify left bottom))
+  )
   (label "mot-l-a1" (at 211.328 42.418 0) (fields_autoplaced)
+    (effects (font (size 1.27 1.27)) (justify left bottom))
+  )
+  (label "c1" (at 50.038 45.72 0) (fields_autoplaced)
     (effects (font (size 1.27 1.27)) (justify left bottom))
   )
@@
     (effects (font (size 1.27 1.27)) (justify left bottom))
   )
+  (label "a1" (at 113.157 24.13 0) (fields_autoplaced)
+    (effects (font (size 1.27 1.27)) (justify left bottom))
+  )
   (label "btn-dn" (at 117.602 80.01 180) (fields_autoplaced)
     (effects (font (size 1.27 1.27)) (justify right bottom))
@@
     (effects (font (size 1.27 1.27)) (justify left bottom))
   )
+  (label "c2" (at 50.038 48.26 0) (fields_autoplaced)
+    (effects (font (size 1.27 1.27)) (justify left bottom))
+  )
   (label "swclk" (at 134.366 62.23 0) (fields_autoplaced)
     (effects (font (size 1.27 1.27)) (justify left bottom))
@@
   )
   (label "dspl-cs" (at 26.543 67.183 0) (fields_autoplaced)
+    (effects (font (size 1.27 1.27)) (justify left bottom))
+  )
+  (label "a2" (at 122.555 31.75 0) (fields_autoplaced)
     (effects (font (size 1.27 1.27)) (justify left bottom))
   )
@@
     (effects (font (size 1.27 1.27)) (justify left bottom))
   )
+  (label "a0" (at 113.157 21.59 0) (fields_autoplaced)
+    (effects (font (size 1.27 1.27)) (justify left bottom))
+  )
