File: hw/car.kicad_pcb (KiCad board)
At the start: 2 copper layers, 45 x 96 mm, 76 parts, among them J1 display, J11 aux-1, J12 aux-2, J13 aux-3, J16 btn, J2 SWD, J31 TYPE-C-31-M-12, J32 batt-out, J51 mot-l-a, J52 mot-l-b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

Commit message: плата - надписи
Connections:
- net Net-(J11-Pin_2) renamed /a0
- net Net-(J11-Pin_3) renamed /a1
- net Net-(J12-Pin_2) renamed /a2
- net Net-(J12-Pin_3) renamed /a3
- net Net-(J12-Pin_4) renamed /a4
- net Net-(J13-Pin_2) renamed /c1
- net Net-(J13-Pin_3) renamed /c2
- net Net-(J13-Pin_4) renamed /c3
Other:
- board text added: "+3v3 A2 A3 A4 GND"
- board text added: "+3v3 gnd swdio swclk"
- board text added: "+hw GND spi-clk spi-mosi spi-miso d-cs d-rst d-dc t-cs t-irq"
- board text added: "GND C3 C2 C1 +3v3"
- board text added: "GND sel rt lt dn up"
Changed lines of the file:
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@@
   (net 29 "/swdio")
   (net 30 "/swclk")
-  (net 31 "Net-(J11-Pin_2)")
-  (net 32 "Net-(J11-Pin_3)")
-  (net 33 "Net-(J12-Pin_2)")
-  (net 34 "Net-(J12-Pin_3)")
-  (net 35 "Net-(J12-Pin_4)")
-  (net 36 "Net-(J13-Pin_2)")
-  (net 37 "Net-(J13-Pin_3)")
-  (net 38 "Net-(J13-Pin_4)")
+  (net 31 "/a0")
+  (net 32 "/a1")
+  (net 33 "/a2")
+  (net 34 "/a3")
+  (net 35 "/a4")
+  (net 36 "/c1")
+  (net 37 "/c2")
+  (net 38 "/c3")
   (net 39 "/btn-up")
   (net 40 "/btn-dn")
@@
       (net 13 "batt-info") (pinfunction "PC0") (pintype "bidirectional"))
     (pad "9" smd roundrect (at -5.675 0.25 270) (size 1.55 0.3) (layers "F.Cu" "F.Paste" "F.Mask") (roundrect_rratio 0.25)
-      (net 36 "Net-(J13-Pin_2)") (pinfunction "PC1") (pintype "bidirectional"))
+      (net 36 "/c1") (pinfunction "PC1") (pintype "bidirectional"))
     (pad "10" smd roundrect (at -5.675 0.75 270) (size 1.55 0.3) (layers "F.Cu" "F.Paste" "F.Mask") (roundrect_rratio 0.25)
-      (net 37 "Net-(J13-Pin_3)") (pinfunction "PC2") (pintype "bidirectional"))
+      (net 37 "/c2") (pinfunction "PC2") (pintype "bidirectional"))
     (pad "11" smd roundrect (at -5.675 1.25 270) (size 1.55 0.3) (layers "F.Cu" "F.Paste" "F.Mask") (roundrect_rratio 0.25)
-      (net 38 "Net-(J13-Pin_4)") (pinfunction "PC3") (pintype "bidirectional"))
+      (net 38 "/c3") (pinfunction "PC3") (pintype "bidirectional"))
     (pad "12" smd roundrect (at -5.675 1.75 270) (size 1.55 0.3) (layers "F.Cu" "F.Paste" "F.Mask") (roundrect_rratio 0.25)
       (net 4 "GND") (pinfunction "VSSA") (pintype "power_in"))
@@
       (net 12 "+3.3VA") (pinfunction "VDDA") (pintype "power_in"))
     (pad "14" smd roundrect (at -5.675 2.75 270) (size 1.55 0.3) (layers "F.Cu" "F.Paste" "F.Mask") (roundrect_rratio 0.25)
-      (net 31 "Net-(J11-Pin_2)") (pinfunction "PA0") (pintype "bidirectional"))
+      (net 31 "/a0") (pinfunction "PA0") (pintype "bidirectional"))
     (pad "15" smd roundrect (at -5.675 3.25 270) (size 1.55 0.3) (layers "F.Cu" "F.Paste" "F.Mask") (roundrect_rratio 0.25)
-      (net 32 "Net-(J11-Pin_3)") (pinfunction "PA1") (pintype "bidirectional"))
+      (net 32 "/a1") (pinfunction "PA1") (pintype "bidirectional"))
     (pad "16" smd roundrect (at -5.675 3.75 270) (size 1.55 0.3) (layers "F.Cu" "F.Paste" "F.Mask") (roundrect_rratio 0.25)
-      (net 33 "Net-(J12-Pin_2)") (pinfunction "PA2") (pintype "bidirectional"))
+      (net 33 "/a2") (pinfunction "PA2") (pintype "bidirectional"))
     (pad "17" smd roundrect (at -3.75 5.675 270) (size 0.3 1.55) (layers "F.Cu" "F.Paste" "F.Mask") (roundrect_rratio 0.25)
-      (net 34 "Net-(J12-Pin_3)") (pinfunction "PA3") (pintype "bidirectional"))
+      (net 34 "/a3") (pinfunction "PA3") (pintype "bidirectional"))
     (pad "18" smd roundrect (at -3.25 5.675 270) (size 0.3 1.55) (layers "F.Cu" "F.Paste" "F.Mask") (roundrect_rratio 0.25)
       (net 4 "GND") (pinfunction "VSS") (pintype "power_in"))
@@
       (net 11 "+3V3") (pinfunction "VDD") (pintype "power_in"))
     (pad "20" smd roundrect (at -2.25 5.675 270) (size 0.3 1.55) (layers "F.Cu" "F.Paste" "F.Mask") (roundrect_rratio 0.25)
-      (net 35 "Net-(J12-Pin_4)") (pinfunction "PA4") (pintype "bidirectional"))
+      (net 35 "/a4") (pinfunction "PA4") (pintype "bidirectional"))
     (pad "21" smd roundrect (at -1.75 5.675 270) (size 0.3 1.55) (layers "F.Cu" "F.Paste" "F.Mask") (roundrect_rratio 0.25)
       (net 28 "/spi-clk") (pinfunction "PA5") (pintype "bidirectional"))
@@
     (property "ki_keywords" "connector")
     (attr through_hole)
-    (fp_text reference "J1" (at 26.5176 1.888 90) (layer "B.SilkS")
+    (fp_text reference "J1" (at 26.2636 -1.541 90) (layer "B.SilkS")
         (effects (font (size 0.7 0.7) (thickness 0.15)) (justify mirror))
     )
-    (fp_text value "display" (at 11.25 -4.6 90) (layer "B.SilkS")
+    (fp_text value "display" (at 27.4066 -2.684 90) (layer "B.SilkS")
         (effects (font (size 0.7 0.7) (thickness 0.15)) (justify mirror))
     )
@@
       (net 11 "+3V3") (pinfunction "Pin_1") (pintype "passive"))
     (pad "2" thru_hole oval (at 2.5 0) (size 1.7 1.95) (drill 0.95) (layers "*.Cu" "*.Mask")
-      (net 31 "Net-(J11-Pin_2)") (pinfunction "Pin_2") (pintype "passive"))
+      (net 31 "/a0") (pinfunction "Pin_2") (pintype "passive"))
     (pad "3" thru_hole oval (at 5 0) (size 1.7 1.95) (drill 0.95) (layers "*.Cu" "*.Mask")
-      (net 32 "Net-(J11-Pin_3)") (pinfunction "Pin_3") (pintype "passive"))
+      (net 32 "/a1") (pinfunction "Pin_3") (pintype "passive"))
     (pad "4" thru_hole oval (at 7.5 0) (size 1.7 1.95) (drill 0.95) (layers "*.Cu" "*.Mask")
       (net 4 "GND") (pinfunction "Pin_4") (pintype "passive"))
@@
         (effects (font (size 0.7 0.7) (thickness 0.15)) (justify mirror))
     )
-    (fp_text value "btn" (at 6.25 -4.6 90) (layer "B.SilkS")
+    (fp_text value "btn" (at -3.4766 -2.286 90) (layer "B.SilkS")
         (effects (font (size 0.7 0.7) (thickness 0.15)) (justify mirror))
     )
@@
         (effects (font (size 0.7 0.7) (thickness 0.15)) (justify mirror))
     )
-    (fp_text value "aux-3" (at 5 -4.6 90) (layer "B.SilkS")
+    (fp_text value "aux-3" (at 14.612 -1.905 90) (layer "B.SilkS")
         (effects (font (size 0.7 0.7) (thickness 0.15)) (justify mirror))
     )
@@
       (net 11 "+3V3") (pinfunction "Pin_1") (pintype "passive"))
     (pad "2" thru_hole oval (at 2.5 0 90) (size 1.7 1.95) (drill 0.95) (layers "*.Cu" "*.Mask")
-      (net 36 "Net-(J13-Pin_2)") (pinfunction "Pin_2") (pintype "passive"))
+      (net 36 "/c1") (pinfunction "Pin_2") (pintype "passive"))
     (pad "3" thru_hole oval (at 5 0 90) (size 1.7 1.95) (drill 0.95) (layers "*.Cu" "*.Mask")
-      (net 37 "Net-(J13-Pin_3)") (pinfunction "Pin_3") (pintype "passive"))
+      (net 37 "/c2") (pinfunction "Pin_3") (pintype "passive"))
     (pad "4" thru_hole oval (at 7.5 0 90) (size 1.7 1.95) (drill 0.95) (layers "*.Cu" "*.Mask")
-      (net 38 "Net-(J13-Pin_4)") (pinfunction "Pin_4") (pintype "passive"))
+      (net 38 "/c3") (pinfunction "Pin_4") (pintype "passive"))
     (pad "5" thru_hole oval (at 10 0 90) (size 1.7 1.95) (drill 0.95) (layers "*.Cu" "*.Mask")
       (net 4 "GND") (pinfunction "Pin_5") (pintype "passive"))
@@
     (property "ki_keywords" "connector")
     (attr through_hole)
-    (fp_text reference "J12" (at -4.3434 -2.811 90) (layer "B.SilkS")
+    (fp_text reference "J12" (at -3.9624 -1.541 90) (layer "B.SilkS")
         (effects (font (size 0.7 0.7) (thickness 0.15)) (justify mirror))
     )
-    (fp_text value "aux-2" (at 5 -4.6 90) (layer "B.SilkS")
+    (fp_text value "aux-2" (at -4.3434 -2.684 90) (layer "B.SilkS")
         (effects (font (size 0.7 0.7) (thickness 0.15)) (justify mirror))
     )
@@
       (net 11 "+3V3") (pinfunction "Pin_1") (pintype "passive"))
     (pad "2" thru_hole oval (at 2.5 0 270) (size 1.7 1.95) (drill 0.95) (layers "*.Cu" "*.Mask")
-      (net 33 "Net-(J12-Pin_2)") (pinfunction "Pin_2") (pintype "passive"))
+      (net 33 "/a2") (pinfunction "Pin_2") (pintype "passive"))
     (pad "3" thru_hole oval (at 5 0 270) (size 1.7 1.95) (drill 0.95) (layers "*.Cu" "*.Mask")
-      (net 34 "Net-(J12-Pin_3)") (pinfunction "Pin_3") (pintype "passive"))
+      (net 34 "/a3") (pinfunction "Pin_3") (pintype "passive"))
     (pad "4" thru_hole oval (at 7.5 0 270) (size 1.7 1.95) (drill 0.95) (layers "*.Cu" "*.Mask")
-      (net 35 "Net-(J12-Pin_4)") (pinfunction "Pin_4") (pintype "passive"))
+      (net 35 "/a4") (pinfunction "Pin_4") (pintype "passive"))
     (pad "5" thru_hole oval (at 10 0 270) (size 1.7 1.95) (drill 0.95) (layers "*.Cu" "*.Mask")
       (net 4 "GND") (pinfunction "Pin_5") (pintype "passive"))
@@
   (gr_line (start 50.8 28.956) (end 50.8 117.856)
     (stroke (width 0.1) (type default)) (layer "Edge.Cuts"))
+  (gr_text "GND\n\nC3\n\nC2\n\nC1\n\n+3v3" (at 88.392 49.149) (layer "B.SilkS")
+    (effects (font (size 0.77 0.8) (thickness 0.18) bold) (justify left bottom mirror))
+  )
+  (gr_text "+hw\n\nGND\n\nspi-clk\n\nspi-mosi\n\nspi-miso\n\nd-cs\n\nd-rst\n\nd-dc\n\nt-cs\n\nt-irq" (at 58.166 78.994) (layer "B.SilkS")
+    (effects (font (size 0.77 0.8) (thickness 0.18) bold) (justify right bottom mirror))
+  )
+  (gr_text "+3v3\ngnd\nswdio\nswclk" (at 89.281 88.265) (layer "B.SilkS")
+    (effects (font (size 0.77 0.8) (thickness 0.18) bold) (justify left bottom mirror))
+  )
+  (gr_text "GND\n\nsel\n\nrt\n\nlt\n\ndn\n\nup" (at 88.392 69.342) (layer "B.SilkS")
+    (effects (font (size 0.77 0.8) (thickness 0.18) bold) (justify left bottom mirror))
+  )
+  (gr_text "+3v3\n\nA2\n\nA3\n\nA4\n\nGND" (at 58.166 49.022) (layer "B.SilkS")
+    (effects (font (size 0.77 0.8) (thickness 0.18) bold) (justify right bottom mirror))
+  )
   (segment (start 63.0428 88.392) (end 62.992 88.519) (width 0.4) (layer "F.Cu") (net 1))
   (segment (start 74.7268 54.864) (end 72.8472 54.864) (width 0.5) (layer "F.Cu") (net 1))

Commit message: плата - небольшие правки
Other:
- board text added: "G a2 a1 +3v3"
